File: KiCAD/MZ-80B_GRAM1.kicad_pcb (KiCad board)
At the start: 2 copper layers, 100 x 160 mm, 50 parts, among them J1 MZ-80B_1, J2 MZ-80B_2, J3 Conn_02x05_Odd_Even, U1 6264, U10 74LS93, U11 74LS93, U12 74LS93, U13 74LS245, U14 74LS165, U15 74LS175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

Commit message: Add files via upload
Other:
- board text removed: "Japanese version"
